File: Hardware/RoombaRio/RoombaRio.kicad_pcb (KiCad board)
At the start: 2 copper layers, 74.5 x 70 mm, 2 parts, among them J101 Raspberry_Pi_2_3, J102 RoombaSerial

Commit message: Inital power mgmnt
Parts:
- added C101: 10uf, Capacitor_SMD:CP_Elec_4x3, F.Cu at (96.8, 16.2)
- added C102: 100nF, Capacitor_SMD:C_0805_2012Metric, F.Cu at (109.0, 23.1)
- added C103: 1uF, Capacitor_SMD:C_0805_2012Metric, F.Cu at (109.0, 19.0)
- added D101: PWR, LED_SMD:LED_0805_2012Metric, F.Cu at (107.1, -30.0)
- added R101: 1K, Resistor_SMD:R_0805_2012Metric, F.Cu at (107.0, -27.0)
- added U101: AMS1117CD, Package_TO_SOT_SMD:TO-252-3_TabPin2, F.Cu at (104.0, 22.0)
Connections:
- net +19V renamed +BATT
- J101 pad 1: unconnected-(J101-3V3-Pad1) -> +3V3
- J101 pad 14: unconnected-(J101-GND-Pad14) -> GND
- J101 pad 17: unconnected-(J101-3V3-Pad17) -> +3V3
- J101 pad 2: unconnected-(J101-5V-Pad2) -> +5V
- J101 pad 20: unconnected-(J101-GND-Pad20) -> GND
- J101 pad 25: unconnected-(J101-GND-Pad25) -> GND
- J101 pad 30: unconnected-(J101-GND-Pad30) -> GND
- J101 pad 34: unconnected-(J101-GND-Pad34) -> GND
- J101 pad 39: unconnected-(J101-GND-Pad39) -> GND
- J101 pad 4: unconnected-(J101-5V-Pad4) -> +5V
- J101 pad 6: unconnected-(J101-GND-Pad6) -> GND
- J101 pad 9: unconnected-(J101-GND-Pad9) -> GND
- J102 pad 3: unconnected-(J102-Pad3) -> /ROOMBA_RX
- J102 pad 4: unconnected-(J102-Pad4) -> /ROOMBA_TX
- J102 pad 5: unconnected-(J102-Pad5) -> /ROOMBA_BRC
Routing:
- added copper zone on B.Cu, net GND
- added copper zone on F.Cu, net GND

Commit message: off to robotics
Parts:
- added J103: i2c Header, Connector_JST:JST_XH_S4B-XH-A_1x04_P2.50mm_Horizontal, F.Cu at (95.8, 25.1)
- added J104: GPIO, Connector_JST:JST_XH_S6B-XH-A_1x06_P2.50mm_Horizontal, F.Cu at (76.8, 25.1)
- added Q101: BSS138, Package_TO_SOT_SMD:SOT-23, F.Cu at (117.1, -3.40)
- added Q102: BSS138, Package_TO_SOT_SMD:SOT-23, F.Cu at (117.1, 1.05)
- added Q103: DNF, Package_TO_SOT_SMD:SOT-23, F.Cu at (117.1, 5.50)
- added R102: 10k, Resistor_SMD:R_0805_2012Metric, F.Cu at (112.4, -4.15)
- added R103: 10k, Resistor_SMD:R_0805_2012Metric, F.Cu at (112.4, -1.20)
- added R104: 10k, Resistor_SMD:R_0805_2012Metric, F.Cu at (112.4, 1.75)
- added R105: 10k, Resistor_SMD:R_0805_2012Metric, F.Cu at (112.4, 4.70)
- added R106: DNF, Resistor_SMD:R_0805_2012Metric, F.Cu at (112.4, 7.65)
- added R107: DNF, Resistor_SMD:R_0805_2012Metric, F.Cu at (112.4, 10.6)
- R101: value 1K -> 2.2K
- moved C102 21.8 mm to (105.5, 1.50), turned to 0 degrees
- moved C103 19.0 mm to (101.5, 1.50), turned to 180 degrees
- moved U101 15.5 mm to (104.5, 6.50), turned to 0 degrees
- moved D101 9.50 mm to (116.6, -30.0)
- moved R101 9.50 mm to (116.5, -27.0)
- moved C101 3.14 mm to (98.7, 13.7), turned to -90 degrees
Connections:
- J101 pad 10: unconnected-(J101-GPIO15/RXD-Pad10) -> /PI_RX
- J101 pad 19: unconnected-(J101-MOSI0/GPIO10-Pad19) -> /GPIO10
- J101 pad 21: unconnected-(J101-MISO0/GPIO9-Pad21) -> /GPIO9
- J101 pad 23: unconnected-(J101-SCLK0/GPIO11-Pad23) -> /GPIO11
- J101 pad 27: unconnected-(J101-ID_SD/GPIO0-Pad27) -> /GPIO0
- J101 pad 28: unconnected-(J101-ID_SC/GPIO1-Pad28) -> /GPIO1
- J101 pad 3: unconnected-(J101-SDA/GPIO2-Pad3) -> /SDA
- J101 pad 5: unconnected-(J101-SCL/GPIO3-Pad5) -> /SCL
- J101 pad 8: unconnected-(J101-GPIO14/TXD-Pad8) -> /PI_TX
Other:
- board text added: "${FULL_REVISION}"
- board text added: "3v3"
- board text added: "GPIO0"
- board text added: "GPIO1"
- board text added: "GPIO10"
- board text added: "GPIO11"
- board text added: "GPIO9"
- board text added: "SCL"
- board text added: "SDA"
